File: lora-testing-board/lora-testing-board.kicad_pcb (KiCad board)
At the start: 2 copper layers, 49.5 x 31.8 mm, 6 parts, among them J1 Conn_01x02_Male, J2 Conn_01x06_Male, J3 U.FL-R-SMT-1_10_, J4 Conn_01x07_Male, U1 RFM95W-915S2

Commit message: Added IDFv3 and Gerber
Parts:
- added REF**: MountingHole_3.2mm_M3, MountingHole:MountingHole_3.2mm_M3, F.Cu at (77.0, 86.0)
- added REF**: MountingHole_3.2mm_M3, MountingHole:MountingHole_3.2mm_M3, F.Cu at (128.0, 86.0)
- added REF**: MountingHole_3.2mm_M3, MountingHole:MountingHole_3.2mm_M3, F.Cu at (128.0, 118.0)
- added REF**: MountingHole_3.2mm_M3, MountingHole:MountingHole_3.2mm_M3, F.Cu at (77.0, 118.0)
Other:
- board size 49.5 x 31.8 mm -> 69 x 50 mm
- board text added: "GPS Testing Board"
- board text added: "Hackaday Dream Team 2021"
- board text added: "L.W. 19-07-2021"
- board text removed: "18-07-2021"
- board text removed: "L.W"
Changed lines of the file:
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@@
   (general
     (thickness 1.6)
-    (drawings 29)
+    (drawings 30)
     (tracks 89)
     (zones 0)
-    (modules 6)
+    (modules 10)
     (nets 15)
   )
@@
   )
   (setup
-    (last_trace_width 0.5)
+    (last_trace_width 0.25)
     (user_trace_width 0.3)
     (user_trace_width 0.5)
@@
     (mod_text_size 1 1)
     (mod_text_width 0.15)
-    (pad_size 1.524 1.524)
-    (pad_drill 0.762)
+    (pad_size 3.2 3.2)
+    (pad_drill 3.2)
     (pad_to_mask_clearance 0)
     (aux_axis_origin 0 0)
-    (visible_elements FFFFFF7F)
+    (visible_elements 7FFFFFFF)
     (pcbplotparams
       (layerselection 0x010fc_ffffffff)
@@
       (usegerberadvancedattributes true)
       (creategerberjobfile true)
-      (excludeedgelayer true)
+      (excludeedgelayer false)
       (linewidth 0.100000)
       (plotframeref false)
       (viasonmask false)
       (mode 1)
-      (useauxorigin false)
+      (useauxorigin true)
       (hpglpennumber 1)
       (hpglpenspeed 20)
@@
       (plotvalue true)
       (plotinvisibletext false)
-      (padsonsilk false)
+      (padsonsilk true)
       (subtractmaskfromsilk false)
       (outputformat 1)
       (mirror false)
-      (drillshape 1)
+      (drillshape 0)
       (scaleselection 1)
-      (outputdirectory ""))
+      (outputdirectory "Gerber/"))
   )
   (net 0 "")
@@
     (add_net "Net-(J4-Pad7)")
   )
+  (module MountingHole:MountingHole_3.2mm_M3 (layer F.Cu)
+    (at 77 86)
+    (descr "Mounting Hole 3.2mm, no annular, M3")
+    (tags "mounting hole 3.2mm no annular m3")
+    (attr virtual)
+    (fp_text reference REF** (at 0 -4.2) (layer F.SilkS)
+      (effects (font (size 1 1) (thickness 0.15)))
+    )
+    (fp_text value MountingHole_3.2mm_M3 (at 0 4.2) (layer F.Fab)
+      (effects (font (size 1 1) (thickness 0.15)))
+    )
+    (fp_circle (center 0 0) (end 3.2 0) (layer Cmts.User) (width 0.15))
+    (fp_circle (center 0 0) (end 3.45 0) (layer F.CrtYd) (width 0.05))
+    (fp_text user %R (at 0.3 0) (layer F.Fab)
+      (effects (font (size 1 1) (thickness 0.15)))
+    )
+    (pad 1 np_thru_hole circle (at 0 0) (size 3.2 3.2) (drill 3.2) (layers *.Cu *.Mask))
+  )
+  (module MountingHole:MountingHole_3.2mm_M3 (layer F.Cu)
+    (at 128 86)
+    (descr "Mounting Hole 3.2mm, no annular, M3")
+    (tags "mounting hole 3.2mm no annular m3")
+    (attr virtual)
+    (fp_text reference REF** (at 0 -4.2) (layer F.SilkS)
+      (effects (font (size 1 1) (thickness 0.15)))
+    )
+    (fp_text value MountingHole_3.2mm_M3 (at 0 4.2) (layer F.Fab)
+      (effects (font (size 1 1) (thickness 0.15)))
+    )
+    (fp_circle (center 0 0) (end 3.45 0) (layer F.CrtYd) (width 0.05))
+    (fp_circle (center 0 0) (end 3.2 0) (layer Cmts.User) (width 0.15))
+    (fp_text user %R (at 0.3 0) (layer F.Fab)
+      (effects (font (size 1 1) (thickness 0.15)))
+    )
+    (pad 1 np_thru_hole circle (at 0 0) (size 3.2 3.2) (drill 3.2) (layers *.Cu *.Mask))
+  )
+  (module MountingHole:MountingHole_3.2mm_M3 (layer F.Cu)
+    (at 128 118)
+    (descr "Mounting Hole 3.2mm, no annular, M3")
+    (tags "mounting hole 3.2mm no annular m3")
+    (attr virtual)
+    (fp_text reference REF** (at 0 -4.2) (layer F.SilkS)
+      (effects (font (size 1 1) (thickness 0.15)))
+    )
+    (fp_text value MountingHole_3.2mm_M3 (at 0 4.2) (layer F.Fab)
+      (effects (font (size 1 1) (thickness 0.15)))
+    )
+    (fp_circle (center 0 0) (end 3.2 0) (layer Cmts.User) (width 0.15))
+    (fp_circle (center 0 0) (end 3.45 0) (layer F.CrtYd) (width 0.05))
+    (fp_text user %R (at 0.3 0) (layer F.Fab)
+      (effects (font (size 1 1) (thickness 0.15)))
+    )
+    (pad 1 np_thru_hole circle (at 0 0) (size 3.2 3.2) (drill 3.2) (layers *.Cu *.Mask))
+  )
+  (module MountingHole:MountingHole_3.2mm_M3 (layer F.Cu)
+    (at 77 118)
+    (descr "Mounting Hole 3.2mm, no annular, M3")
+    (tags "mounting hole 3.2mm no annular m3")
+    (attr virtual)
+    (fp_text reference REF** (at 0 -4.2) (layer F.SilkS)
+      (effects (font (size 1 1) (thickness 0.15)))
+    )
+    (fp_text value MountingHole_3.2mm_M3 (at 0 4.2) (layer F.Fab)
+      (effects (font (size 1 1) (thickness 0.15)))
+    )
+    (fp_circle (center 0 0) (end 3.45 0) (layer F.CrtYd) (width 0.05))
+    (fp_circle (center 0 0) (end 3.2 0) (layer Cmts.User) (width 0.15))
+    (fp_text user %R (at 0.3 0) (layer F.Fab)
+      (effects (font (size 1 1) (thickness 0.15)))
+    )
+    (pad 1 np_thru_hole circle (at 0 0) (size 3.2 3.2) (drill 3.2) (layers *.Cu *.Mask))
+  )
   (module Capacitor_SMD:C_0805_2012Metric (layer F.Cu)
     (at 92.71 89.85 270)
@@
     (pad 1 smd rect (at -1.475 0 90) (size 1.05 2.2) (layers F.Cu F.Paste F.Mask)
       (net 2 GND1))
-    (model U.FL-R-SMT-1_10_.stp
-      (offset (xyz 0 0.04999999999413419 0))
+    (model ${KIPRJMOD}/3D/U.FL-R-SMT-1_10_.stp
+      (at (xyz 0 0 0))
       (scale (xyz 1 1 1))
       (rotate (xyz 0 0 0))
@@
       (rotate (xyz 0 0 0))
     )
-  )
-  (gr_text 18-07-2021 (at 118.11 90.424) (layer F.SilkS)
-    (effects (font (size 1 1) (thickness 0.15)) (justify right))
-  )
-  (gr_text L.W (at 118.11 88.392) (layer F.SilkS)
-    (effects (font (size 1 1) (thickness 0.15)) (justify right))
-  )
-  (gr_line (start 128.27 83.82) (end 81.28 83.82) (layer Edge.Cuts) (width 0.05))
-  (gr_line (start 129.54 114.3) (end 129.54 85.09) (layer Edge.Cuts) (width 0.05))
-  (gr_line (start 81.28 115.57) (end 128.27 115.57) (layer Edge.Cuts) (width 0.05))
-  (gr_line (start 80.01 85.09) (end 80.01 114.3) (layer Edge.Cuts) (width 0.05))
+    (model "${KIPRJMOD}/3D/RFM95 LoRa v15.step"
+      (offset (xyz 8 -8 0))
+      (scale (xyz 1 1 1))
+      (rotate (xyz 90 180 0))
+    )
+  )
+  (gr_arc (start 128 118) (end 128 127) (angle -90) (layer Edge.Cuts) (width 0.05))
+  (gr_arc (start 77 118) (end 68 118) (angle -90) (layer Edge.Cuts) (width 0.05))
+  (gr_arc (start 128 86) (end 137 86) (angle -90) (layer Edge.Cuts) (width 0.05))
+  (gr_arc (start 77 86) (end 77 77) (angle -90) (layer Edge.Cuts) (width 0.05))
+  (gr_text "GPS Testing Board" (at 81.407 81.5594) (layer F.SilkS)
+    (effects (font (size 1.5 1.5) (thickness 0.3)) (justify left))
+  )
+  (gr_text "L.W.      19-07-2021" (at 81.5594 83.7438) (layer F.SilkS)
+    (effects (font (size 1.5 1.5) (thickness 0.3)) (justify left))
+  )
+  (gr_text "Hackaday Dream Team 2021" (at 81.534 79.502) (layer F.SilkS)
+    (effects (font (size 1.5 1.5) (thickness 0.3)) (justify left))
+  )
+  (gr_line (start 128 77) (end 77 77) (layer Edge.Cuts) (width 0.05))
+  (gr_line (start 137 118) (end 137 86) (layer Edge.Cuts) (width 0.05))
+  (gr_line (start 77 127) (end 128 127) (layer Edge.Cuts) (width 0.05))
+  (gr_line (start 68 86) (end 68 118) (layer Edge.Cuts) (width 0.05))
   (gr_text MOSI (at 86.36 100.33) (layer F.SilkS)
     (effects (font (size 1.5 1.5) (thickness 0.3)) (justify right))
   )
-  (gr_arc (start 81.28 114.3) (end 80.01 114.3) (angle -90) (layer Edge.Cuts) (width 0.05))
-  (gr_arc (start 81.28 85.09) (end 81.28 83.82) (angle -90) (layer Edge.Cuts) (width 0.05))
-  (gr_arc (start 128.27 85.09) (end 129.54 85.09) (angle -90) (layer Edge.Cuts) (width 0.05))
-  (gr_arc (start 128.27 114.3) (end 128.27 115.57) (angle -90) (layer Edge.Cuts) (width 0.05))
-  (gr_text RFM95W-915S2 (at 105.156 85.598) (layer F.SilkS)
+  (gr_text RFM95W-915S2 (at 104.267 91.7956) (layer F.SilkS)
     (effects (font (size 1.5 1.5) (thickness 0.3)))
   )
@@
     (effects (font (size 1.5 1.5) (thickness 0.3)) (justify right))
   )
-  (gr_text GND (at 86.36 91.44) (layer F.SilkS)
-    (effects (font (size 1.5 1.5) (thickness 0.3)) (justify right))
-  )
+  (gr_text GND (at 86.4362 91.3638) (layer F.SilkS)
+    (effects (font (size 1.5 1.5) (thickness 0.3)) (justify right))
+  )

Commit message: Updated schematic, gerbers and added README
Other:
- board text added: "LoRa Testing Board v1.0"
- board text removed: "GPS Testing Board"
