File: lora-testing-board/lora-testing-board.sch (KiCad schematic (older format))
At the start: 6 parts

Commit message: Added PCB for RFM95W-915S2
Parts:
- removed C?: CAP, symbol pspice:CAP
- removed J?: U.FL-R-SMT-1_10_, U.FL-R-SMT-1(10), symbol U.FL-R-SMT-1_10_:U.FL-R-SMT-1_10_
- added C1: C-10uF-0805, Capacitor_SMD:C_0805_2012Metric, symbol C-10uF-0805:C-10uF-0805
- added J3: U.FL-R-SMT-1_10_, U.FL-R-SMT-1(10):U.FL-R-SMT-1_10_, symbol U.FL-R-SMT-1_10_:U.FL-R-SMT-1_10_
- J1: renamed from J?; footprint (none) -> Connector_PinSocket_2.54mm:PinSocket_1x02_P2.54mm_Vertical
- J2: renamed from J?; footprint (none) -> Connector_PinSocket_2.54mm:PinSocket_1x06_P2.54mm_Vertical
- J4: renamed from J?; footprint (none) -> Connector_PinSocket_2.54mm:PinSocket_1x07_P2.54mm_Vertical
- U1: renamed from U?; footprint (none) -> RF_Module:HOPERF_RFM9XW_SMD; symbol RF_Module:RFM95W-915S2 -> RFM95W-915S2:RFM95W-915S2; Supplier 1 (none) -> Digi-Key; Supplier Part Number 1 (none) -> RFM95W-915S2-ND
Connections:
- net GND1: now also J1.1 (Pin_1), J2.1 (Pin_1), J4.1 (Pin_1), C1.2, J3.1, J3.2; no longer J1.2 (Pin_2), J2.6 (Pin_6), J4.7 (Pin_7)
- net at U1.11 (DIO3): now also J4.5 (Pin_5); no longer J4.3 (Pin_3)
- net at U1.12 (DIO4): now also J4.6 (Pin_6); no longer J4.2 (Pin_2)
- net at U1.13 (3.3V): now also J1.2 (Pin_2), C1.1; no longer J1.1 (Pin_1)
- net at U1.14 (DIO0): now also J4.2 (Pin_2); no longer J4.6 (Pin_6)
- net at U1.15 (DIO1): now also J4.3 (Pin_3); no longer J4.5 (Pin_5)
- net at U1.2 (MISO): now also J2.6 (Pin_6); no longer J2.3 (Pin_3)
- net at U1.3 (MOSI): now also J2.5 (Pin_5); no longer J2.2 (Pin_2)
- net at U1.4 (SCK): now also J2.4 (Pin_4); no longer J2.1 (Pin_1)
- net at U1.5 (NSS): now also J2.3 (Pin_3); no longer J2.4 (Pin_4)
- net at U1.6 (RESET): now also J2.2 (Pin_2); no longer J2.5 (Pin_5)
- net at U1.7 (DIO5): now also J4.7 (Pin_7); no longer J4.1 (Pin_1)
- net at U1.9 (ANT): now also J3.3
Other:
- note added: "RFM95W-915S2"
- note added: "RST"
- note removed: "RESET"
- note removed: "RFM95W"
Changed lines of the file:
@@
 $EndDescr
 $Comp
-L RF_Module:RFM95W-915S2 U?
+L RFM95W-915S2:RFM95W-915S2 U1
 U 1 1 60F3A12A
 P 6250 4050
-F 0 "U?" H 6250 4731 50  0000 C CNN
+F 0 "U1" H 6250 4731 50  0000 C CNN
 F 1 "RFM95W-915S2" H 6250 4640 50  0000 C CNN
-F 2 "" H 2950 5700 50  0001 C CNN
-F 3 "https://www.hoperf.com/data/upload/portal/20181127/5bfcbea20e9ef.pdf" H 2950 5700 50  0001 C CNN
+F 2 "RF_Module:HOPERF_RFM9XW_SMD" H 2950 5700 50  0001 C CNN
+F 3 "https://www.rfsolutions.co.uk/downloads/1463993415RFM95_96_97_98W.pdf" H 2950 5700 50  0001 C CNN
+F 4 "Digi-Key" H 6250 4050 50  0001 C CNN "Supplier 1"
+F 5 "RFM95W-915S2-ND" H 6250 4050 50  0001 C CNN "Supplier Part Number 1"
 	1    6250 4050
 	1    0    0    -1
 $EndComp
 $Comp
-L Connector:Conn_01x06_Male J?
+L Connector:Conn_01x06_Male J2
 U 1 1 60F3E586
-P 4450 3950
-F 0 "J?" H 4558 4331 50  0000 C CNN
-F 1 "Conn_01x06_Male" H 4558 4240 50  0000 C CNN
-F 2 "" H 4450 3950 50  0001 C CNN
-F 3 "~" H 4450 3950 50  0001 C CNN
-	1    4450 3950
-	1    0    0    -1
+P 4450 4050
+F 0 "J2" H 4550 3550 50  0000 C CNN
+F 1 "Conn_01x06_Male" H 4550 3650 50  0000 C CNN
+F 2 "Connector_PinSocket_2.54mm:PinSocket_1x06_P2.54mm_Vertical" H 4450 4050 50  0001 C CNN
+F 3 "~" H 4450 4050 50  0001 C CNN
+	1    4450 4050
+	1    0    0    1
 $EndComp
 Wire Wire Line
@@
 	5700 4250 5700 4150
 $Comp
-L power:GND1 #PWR?
+L power:GND1 #PWR0101
 U 1 1 60F43691
 P 4800 4300
-F 0 "#PWR?" H 4800 4050 50  0001 C CNN
+F 0 "#PWR0101" H 4800 4050 50  0001 C CNN
 F 1 "GND1" H 4805 4127 50  0000 C CNN
 F 2 "" H 4800 4300 50  0001 C CNN
@@
 	4800 4300 4800 4250
 $Comp
-L power:GND1 #PWR?
+L power:GND1 #PWR0102
 U 1 1 60F43F3C
 P 6250 4750
-F 0 "#PWR?" H 6250 4500 50  0001 C CNN
+F 0 "#PWR0102" H 6250 4500 50  0001 C CNN
 F 1 "GND1" H 6255 4577 50  0000 C CNN
 F 2 "" H 6250 4750 50  0001 C CNN
@@
 	6150 4700 6250 4700
 $Comp
-L Connector:Conn_01x02_Male J?
+L Connector:Conn_01x02_Male J1
 U 1 1 60F44B42
-P 4450 2950
-F 0 "J?" H 4558 3131 50  0000 C CNN
-F 1 "Conn_01x02_Male" H 4558 3040 50  0000 C CNN
-F 2 "" H 4450 2950 50  0001 C CNN
-F 3 "~" H 4450 2950 50  0001 C CNN
-	1    4450 2950
-	1    0    0    -1
+P 4450 3050
+F 0 "J1" H 4550 2750 50  0000 C CNN
+F 1 "Conn_01x02_Male" H 4550 2850 50  0000 C CNN
+F 2 "Connector_PinSocket_2.54mm:PinSocket_1x02_P2.54mm_Vertical" H 4450 3050 50  0001 C CNN
+F 3 "~" H 4450 3050 50  0001 C CNN
+	1    4450 3050
+	1    0    0    1
 $EndComp
 Wire Wire Line
 	6250 3550 6250 2950
-Wire Wire Line
-	6250 2950 5300 2950
-$Comp
-L power:GND1 #PWR?
+$Comp
+L power:GND1 #PWR0103
 U 1 1 60F45983
 P 4700 3100
-F 0 "#PWR?" H 4700 2850 50  0001 C CNN
+F 0 "#PWR0103" H 4700 2850 50  0001 C CNN
 F 1 "GND1" H 4705 2927 50  0000 C CNN
 F 2 "" H 4700 3100 50  0001 C CNN
@@
 Text Notes 4000 3100 0    50   ~ 0
 GND
-Text Notes 4150 3800 2    50   ~ 0
+Text Notes 4150 4000 2    50   ~ 0
 SCK
 Text Notes 4150 3900 2    50   ~ 0
 MOSI
-Text Notes 4150 4000 2    50   ~ 0
+Text Notes 4150 3800 2    50   ~ 0
 MISO
 Text Notes 4150 4100 2    50   ~ 0
 CS
 Text Notes 4150 4200 2    50   ~ 0
-RESET
+RST
 Text Notes 4150 4300 2    50   ~ 0
 GND
 $Comp
-L pspice:CAP C?
-U 1 1 60F4B157
-P 5300 3200
-F 0 "C?" H 5478 3246 50  0000 L CNN
-F 1 "CAP" H 5478 3155 50  0000 L CNN
-F 2 "" H 5300 3200 50  0001 C CNN
-F 3 "~" H 5300 3200 50  0001 C CNN
-	1    5300 3200
-	1    0    0    -1
-$EndComp
-Connection ~ 5300 2950
-Wire Wire Line
-	5300 2950 4650 2950
-$Comp
-L power:GND1 #PWR?
+L power:GND1 #PWR0104
 U 1 1 60F4C28B
-P 5300 3500
-F 0 "#PWR?" H 5300 3250 50  0001 C CNN
-F 1 "GND1" H 5305 3327 50  0000 C CNN
-F 2 "" H 5300 3500 50  0001 C CNN
-F 3 "" H 5300 3500 50  0001 C CNN
-	1    5300 3500
-	1    0    0    -1
-$EndComp
-Wire Wire Line
-	5300 3500 5300 3450
-$Comp
-L Connector:Conn_01x07_Male J?
+P 5300 3350
+F 0 "#PWR0104" H 5300 3100 50  0001 C CNN
+F 1 "GND1" H 5305 3177 50  0000 C CNN
+F 2 "" H 5300 3350 50  0001 C CNN
+F 3 "" H 5300 3350 50  0001 C CNN
+	1    5300 3350
+	1    0    0    -1
+$EndComp
+$Comp
+L Connector:Conn_01x07_Male J4
 U 1 1 60F51643
 P 7550 4250
-F 0 "J?" H 7700 4750 50  0000 R CNN
-F 1 "Conn_01x07_Male" H 7900 4650 50  0000 R CNN
-F 2 "" H 7550 4250 50  0001 C CNN
+F 0 "J4" H 7700 3750 50  0000 R CNN
+F 1 "Conn_01x07_Male" H 7950 3850 50  0000 R CNN
+F 2 "Connector_PinSocket_2.54mm:PinSocket_1x07_P2.54mm_Vertical" H 7550 4250 50  0001 C CNN
 F 3 "~" H 7550 4250 50  0001 C CNN
 	1    7550 4250
-	-1   0    0    -1
+	-1   0    0    1
 $EndComp
 Wire Wire Line
@@
 	6750 4450 7350 4450
 $Comp
-L power:GND1 #PWR?
+L power:GND1 #PWR0105
 U 1 1 60F55D88
 P 7250 4600
-F 0 "#PWR?" H 7250 4350 50  0001 C CNN
+F 0 "#PWR0105" H 7250 4350 50  0001 C CNN
 F 1 "GND1" H 7255 4427 50  0000 C CNN
 F 2 "" H 7250 4600 50  0001 C CNN
@@
 Wire Notes Line style solid
 	8150 2600 3750 2600
-$Comp
-L U.FL-R-SMT-1_10_:U.FL-R-SMT-1_10_ J?
-U 1 1 60F7CD8D
-P 7100 3200
-F 0 "J?" H 7450 3500 50  0000 L CNN
-F 1 "U.FL-R-SMT-1_10_" H 7150 3400 50  0000 L CNN
-F 2 "U.FL-R-SMT-1(10)" H 7750 3300 50  0001 L CNN
-F 3 "https://www.hirose.com/product/document?clcode=CL0331-0472-2-10&productname=U.FL-R-SMT-1(10)&series=U.FL&documenttype=2DDrawing&lang=en&documentid=0000940684" H 7750 3200 50  0001 L CNN
-F 4 "UFL SMT PCB receptable,DC-6GHz Hirose Straight 50 Surface Mount UFL Connector, Receptacle, Solder Termination Coaxial" H 7750 3100 50  0001 L CNN "Description"
-F 5 "Hirose" H 7750 2900 50  0001 L CNN "Manufacturer_Name"
-F 6 "U.FL-R-SMT-1(10)" H 7750 2800 50  0001 L CNN "Manufacturer_Part_Number"
-F 7 "798-U.FL-R-SMT-110" H 7750 2700 50  0001 L CNN "Mouser Part Number"
-F 8 "https://www.mouser.co.uk/ProductDetail/Hirose-Connector/UFL-R-SMT-110?qs=kL1ClTr6oBoOdtqlGQpQrQ%3D%3D" H 7750 2600 50  0001 L CNN "Mouser Price/Stock"
-F 9 "U.FL-R-SMT-1(10)" H 7750 2500 50  0001 L CNN "Arrow Part Number"
-F 10 "https://www.arrow.com/en/products/u.fl-r-smt-1-10/hirose-electric" H 7750 2400 50  0001 L CNN "Arrow Price/Stock"
-	1    7100 3200
-	1    0    0    -1
-$EndComp
 Wire Wire Line
 	7100 3300 6850 3300
@@
 	6850 3750 6750 3750
 $Comp
-L power:GND1 #PWR?
+L power:GND1 #PWR0106
 U 1 1 60F7F510
 P 7000 3450
-F 0 "#PWR?" H 7000 3200 50  0001 C CNN
+F 0 "#PWR0106" H 7000 3200 50  0001 C CNN
 F 1 "GND1" H 7005 3277 50  0000 C CNN
 F 2 "" H 7000 3450 50  0001 C CNN
@@
 	7000 3400 7000 3450
 Text Notes 8000 2800 2    100  ~ 0
-RFM95W
+RFM95W-915S2
+Wire Wire Line
+	4650 2950 5300 2950
+Wire Wire Line
+	5300 3000 5300 2950
+Connection ~ 5300 2950
+Wire Wire Line
+	5300 2950 6250 2950
+Wire Wire Line
+	5300 3300 5300 3350
+$Comp
+L C-10uF-0805:C-10uF-0805 C1
+U 1 1 60F514A5
+P 5300 3150
+F 0 "C1" H 5415 3150 50  0000 L CNN
+F 1 "C-10uF-0805" H 5800 3250 50  0001 C CNN
+F 2 "Capacitor_SMD:C_0805_2012Metric" H 6150 2950 50  0001 C CNN
+F 3 "" H 5300 3150 50  0001 C CNN
+F 4 "Digi-Key" H 5700 3150 50  0001 C CNN "Supplier 1"
+F 5 "1276-2404-1-ND" H 6300 3150 50  0001 C CNN "Supplier Part Number 1"
+F 6 "Samsung Electro-Mechanics" H 6050 3050 50  0001 C CNN "Manufacturer"
+F 7 "CL21A106KQCLNNC" H 7050 3050 50  0001 C CNN "Manufacturer Part Number"
+	1    5300 3150
+	1    0    0    -1
+$EndComp
+$Comp
+L U.FL-R-SMT-1_10_:U.FL-R-SMT-1_10_ J3
+U 1 1 60F52CF6
+P 7100 3200
+F 0 "J3" H 7400 3450 50  0000 L CNN
+F 1 "U.FL-R-SMT-1_10_" H 7300 3350 50  0000 L CNN
+F 2 "U.FL-R-SMT-1(10):U.FL-R-SMT-1_10_" H 7750 3300 50  0001 L CNN
+F 3 "https://www.hirose.com/product/document?clcode=CL0331-0472-2-10&productname=U.FL-R-SMT-1(10)&series=U.FL&documenttype=2DDrawing&lang=en&documentid=0000940684" H 7750 3200 50  0001 L CNN
+F 4 "UFL SMT PCB receptable,DC-6GHz Hirose Straight 50 Surface Mount UFL Connector, Receptacle, Solder Termination Coaxial" H 7750 3100 50  0001 L CNN "Description"
+F 5 "Hirose" H 7750 2900 50  0001 L CNN "Manufacturer Name"
+F 6 "U.FL-R-SMT-1(10)" H 7750 2800 50  0001 L CNN "Manufacturer Part Number"
+F 7 "798-U.FL-R-SMT-110" H 7750 2700 50  0001 L CNN "Supplier Part Number 2"
+F 8 "Mouser" H 7750 2600 50  0001 L CNN "Supplier 2"
+F 9 "Digi-Key" H 7750 2500 50  0001 L CNN "Supplier 1"
+F 10 "H11891CT-ND" H 7750 2400 50  0001 L CNN "Supplier Part Number 1"
+	1    7100 3200
+	1    0    0    -1
+$EndComp
 $EndSCHEMATC

Commit message: Updated schematic, gerbers and added README
Parts:
- C1: value C-10uF-0805 -> 10uF; symbol C-10uF-0805:C-10uF-0805 -> C-10uF-0805:10uF
Changed lines of the file:
@@
 	5300 3300 5300 3350
 $Comp
-L C-10uF-0805:C-10uF-0805 C1
+L C-10uF-0805:10uF C1
 U 1 1 60F514A5
 P 5300 3150
 F 0 "C1" H 5415 3150 50  0000 L CNN
-F 1 "C-10uF-0805" H 5800 3250 50  0001 C CNN
+F 1 "10uF" H 5510 3070 50  0000 C CNN
 F 2 "Capacitor_SMD:C_0805_2012Metric" H 6150 2950 50  0001 C CNN
 F 3 "" H 5300 3150 50  0001 C CNN
